File: board/Pixel.kicad_pcb (KiCad board)
At the start: 2 copper layers, 106.2 x 57.8 mm, 31 parts, among them J0 Batt+, J1 Batt-, SW0 Reset, SW1 Up, SW2 Down, SW3 Left, SW4 Right, SW5 BTN A, SW6 BTN B, SW7 BTN C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

Commit message: rotated reset diode
Parts:
- moved D0 7.50 mm to (198.2, 46.5), turned to 90 degrees
Connections:
- D0 pad 1: Net-(C1-Pad1) -> Net-(D0-Pad1)
- D0 pad 2: Net-(D0-Pad2) -> Net-(C1-Pad1)
- SW0 pad 2: Net-(D0-Pad2) -> Net-(D0-Pad1)
- U1 pad 1: Net-(D0-Pad2) -> Net-(D0-Pad1)
Routing:
- net Net-(D0-Pad2): track 7.29 -> 0.00 mm
- net Net-(D0-Pad1): track 0.00 -> 6.99 mm
- net Net-(C1-Pad1): track 54.1 -> 54.7 mm

Commit message: fixed connections
Routing:
- net Net-(LS1-Pad1): track 0.00 -> 71.9 mm
- net Net-(R1-Pad1): track 72.8 -> 119.2 mm
- net Net-(U1-Pad6): track 0.00 -> 44.9 mm
- net Net-(U1-Pad7): track 0.00 -> 41.4 mm
- added copper zone on B.Cu, net +5V
- added copper zone on F.Cu, net GND
Changed lines of the file:
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@@
   (general
     (links 71)
-    (no_connects 44)
-    (area 121.856959 34.842055 228.171381 92.785148)
+    (no_connects 10)
+    (area 121.856959 34.842055 228.171381 93.045001)
     (thickness 1.6)
     (drawings 277)
-    (tracks 60)
+    (tracks 80)
     (zones 0)
     (modules 31)
@@
   (segment (start 182.5 39) (end 177.49 44.01) (width 0.25) (layer F.Cu) (net 6))
   (segment (start 159.5 40) (end 159.5 46.5) (width 0.25) (layer F.Cu) (net 7))
+  (segment (start 214.88 43.88) (end 214.13 43.88) (width 0.25) (layer F.Cu) (net 8) (status C00000))
+  (segment (start 214.13 43.88) (end 211.75 41.5) (width 0.25) (layer F.Cu) (net 8) (status 400000))
+  (segment (start 211.75 41.5) (end 204 41.5) (width 0.25) (layer F.Cu) (net 8))
+  (segment (start 204 41.5) (end 199.25 36.75) (width 0.25) (layer F.Cu) (net 8))
+  (segment (start 199.25 36.75) (end 181.25 36.75) (width 0.25) (layer F.Cu) (net 8))
+  (segment (start 181.25 36.75) (end 169.25 48.75) (width 0.25) (layer F.Cu) (net 8))
+  (segment (start 169.25 48.75) (end 154.75 48.75) (width 0.25) (layer F.Cu) (net 8))
+  (segment (start 154.75 48.75) (end 152 46) (width 0.25) (layer F.Cu) (net 8) (status 800000))
   (segment (start 144.4 46) (end 144.4 45.9) (width 0.25) (layer F.Cu) (net 9))
   (segment (start 144.4 45.9) (end 142.04 43.54) (width 0.25) (layer F.Cu) (net 9))
   (segment (start 142.04 43.54) (end 136.62 43.54) (width 0.25) (layer F.Cu) (net 9))
+  (segment (start 194 61.16) (end 195.66 61.16) (width 0.25) (layer F.Cu) (net 10))
+  (segment (start 225.25 49.17) (end 222.5 46.42) (width 0.25) (layer F.Cu) (net 10))
+  (segment (start 225.25 58.5) (end 225.25 49.17) (width 0.25) (layer F.Cu) (net 10))
+  (segment (start 221.5 62.25) (end 225.25 58.5) (width 0.25) (layer F.Cu) (net 10))
+  (segment (start 196.75 62.25) (end 221.5 62.25) (width 0.25) (layer F.Cu) (net 10))
+  (segment (start 195.66 61.16) (end 196.75 62.25) (width 0.25) (layer F.Cu) (net 10))
   (segment (start 189.5 73.5) (end 189.5 65.66) (width 0.25) (layer F.Cu) (net 10))
   (segment (start 189.5 65.66) (end 194 61.16) (width 0.25) (layer F.Cu) (net 10))
@@
   (segment (start 136.62 46.08) (end 136.62 47.62) (width 0.25) (layer F.Cu) (net 18))
   (segment (start 136.62 47.62) (end 151 62) (width 0.25) (layer F.Cu) (net 18))
+  (segment (start 214.88 46.42) (end 201.83 46.42) (width 0.25) (layer B.Cu) (net 19))
+  (segment (start 176.74 48.25) (end 172.49 52.5) (width 0.25) (layer B.Cu) (net 19))
+  (segment (start 200 48.25) (end 176.74 48.25) (width 0.25) (layer B.Cu) (net 19))
+  (segment (start 201.83 46.42) (end 200 48.25) (width 0.25) (layer B.Cu) (net 19))
+  (segment (start 214.88 48.96) (end 178.53 48.96) (width 0.25) (layer B.Cu) (net 20))
+  (segment (start 178.53 48.96) (end 174.99 52.5) (width 0.25) (layer B.Cu) (net 20))
   (segment (start 136.62 41) (end 145 41) (width 0.25) (layer F.Cu) (net 21))
   (segment (start 168 63.5) (end 168 68) (width 0.25) (layer F.Cu) (net 21))
@@
   (segment (start 201.25 43.5) (end 198.25 46.5) (width 0.25) (layer F.Cu) (net 24))
   (segment (start 204 43.5) (end 201.25 43.5) (width 0.25) (layer F.Cu) (net 24))
+  (zone (net 4) (net_name GND) (layer F.Cu) (hatch edge 0.508)
+    (connect_pads (clearance 0.508))
+    (min_thickness 0.254)
+    (fill yes (arc_segments 16) (thermal_gap 0.508) (thermal_bridge_width 0.508))
+    (polygon
+      (pts
+        (xy 232.75 98.5) (xy 118 98.5) (xy 118 29.75) (xy 232.75 29.75)
+      )
+    )
+  )
+  (zone (net 5) (net_name +5V) (layer B.Cu) (hatch edge 0.508)
+    (connect_pads (clearance 0.508))
+    (min_thickness 0.254)
+    (fill yes (arc_segments 16) (thermal_gap 0.508) (thermal_bridge_width 0.508))
+    (polygon
+      (pts
+        (xy 233.75 97.25) (xy 115.25 97.25) (xy 115.25 31.5) (xy 233.75 31.5)
+      )
+    )
+  )
 )
