File: board/Mage.sch (KiCad schematic (older format))
At the start: 31 parts, among them J0 Batt+, J1 Batt-, SW0 Reset, SW1 Up, SW2 Down, SW3 Left, SW4 Right, SW5 BTN A, SW6 BTN B, SW7 BTN C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

Commit message: New, smaller PCB
Parts:
- removed BT1: Lipo, Custom Footprints:4056E_LiIon_loader, symbol Lipo
- removed D2: Power, LEDs:LED_D5.0mm, symbol LED_ALT
- removed J0: Batt+, SMD_Packages:1Pin, symbol Conn_01x01
- removed J1: Batt-, SMD_Packages:1Pin, symbol Conn_01x01
- removed R0: 1K, Resistors_THT:R_Axial_DIN0207_L6.3mm_D2.5mm_P10.16mm_Horizontal, symbol R
- removed R8: 270R, Resistors_THT:R_Axial_DIN0207_L6.3mm_D2.5mm_P10.16mm_Horizontal, symbol R
- removed SW8: PWR MUT PAUS, Buttons_Switches_THT:SW_DIP_x3_W7.62mm_Slide, symbol SW_DIP_x03
- added BT1: Battery_Cell, Custom Footprints:3008_coin_cell, symbol Battery_Cell
- added SW8: POWER, Buttons_Switches_THT:SW_DIP_x1_W7.62mm_Slide, symbol SW_DIP_x01
- R1, R10, R2, R3, R5, R6, R7, R9: footprint Resistors_THT:R_Axial_DIN0207_L6.3mm_D2.5mm_P10.16mm_Horizontal -> Resistors_THT:R_Axial_DIN0207_L6.3mm_D2.5mm_P7.62mm_Horizontal
- R4: value 51k -> 62k; footprint Resistors_THT:R_Axial_DIN0207_L6.3mm_D2.5mm_P10.16mm_Horizontal -> Resistors_THT:R_Axial_DIN0207_L6.3mm_D2.5mm_P7.62mm_Horizontal
Connections:
- net GND: now also LS1.2, BT1.2 (-)
- net +5V renamed +3V3
- net +3V3: now also SW8.2
- new net: BT1.1 (+), SW8.1
Other:
- moved on the sheet: LS1

Commit message: reworked board to make it neater
Added decoupling capacitor for OLED
Removed CR2032, replaced with Lipo
Tweaked layout
Parts:
- removed D0: D_ALT, Diodes_THT:D_A-405_P7.62mm_Horizontal, symbol D_ALT
- added C2: 0.1uF, Capacitors_THT:C_Rect_L7.0mm_W2.5mm_P5.00mm, symbol C
- BT1: value Battery_Cell -> 3.7v Lipo; footprint Custom Footprints:3008_coin_cell -> Custom Footprints:LiPo_Pads
- C0: renamed from C1; value 0.1uF -> 1.0uF; footprint Capacitors_THT:CP_Radial_Tantal_D5.0mm_P5.00mm -> Capacitors_THT:C_Rect_L7.0mm_W2.5mm_P5.00mm
- C1: renamed from C0; value 100nF -> 0.1uF; footprint Capacitors_THT:CP_Radial_Tantal_D5.0mm_P5.00mm -> Capacitors_THT:C_Rect_L7.0mm_W2.5mm_P5.00mm
- R4: value 62k -> 68k
- SW5: value BTN A -> A
- SW6: value BTN B -> B
- SW7: value BTN C -> C
- renumbered D1 to D0
Connections:
- net +3V3: now also C2.2
- net GND: now also C2.1
- net at SW0.2, U1.1 (RST_ADC0): now also C0.1, D0.2 (A), R10.2, U2.5 (RESET)

Commit message: updated board to KiCAD 5.0
Parts:
- BT1: symbol Battery_Cell -> Device:Battery_Cell
- C0, C1, C2: symbol C -> Device:C
- D0: symbol D_ALT -> Device:D_ALT
- LS1: symbol Speaker -> Device:Speaker
- R1, R10, R2, R3, R4, R5, R6, R7, R9: symbol R -> Device:R
- SW0, SW1, SW2, SW3, SW4, SW5, SW6, SW7: symbol SW_Push -> switches:SW_Push
- SW8: symbol SW_DIP_x01 -> switches:SW_DIP_x01
- U1: footprint Housings_DIP:DIP-8_W7.62mm_Socket -> Housings_QFP:TQFP-44_10x10mm_Pitch0.8mm; symbol ATTiny85 -> Custom-Library:ATTiny85
- U2: symbol SSD1306_OLED -> Custom-Library:SSD1306_OLED
Changed lines of the file:
@@
-EESchema Schematic File Version 2
-LIBS:power
-LIBS:device
-LIBS:switches
-LIBS:relays
-LIBS:motors
-LIBS:transistors
-LIBS:conn
-LIBS:linear
-LIBS:regul
-LIBS:74xx
-LIBS:cmos4000
-LIBS:adc-dac
-LIBS:memory
-LIBS:xilinx
-LIBS:microcontrollers
-LIBS:dsp
-LIBS:microchip
-LIBS:analog_switches
-LIBS:motorola
-LIBS:texas
-LIBS:intel
-LIBS:audio
-LIBS:interface
-LIBS:digital-audio
-LIBS:philips
-LIBS:display
-LIBS:cypress
-LIBS:siliconi
-LIBS:opto
-LIBS:atmel
-LIBS:contrib
-LIBS:valves
-LIBS:Custom Library
+EESchema Schematic File Version 4
 LIBS:Mage-cache
-EELAYER 25 0
+EELAYER 26 0
 EELAYER END
 $Descr A4 11693 8268
@@
 $EndDescr
 $Comp
-L ATTiny85 U1
+L Custom-Library:ATTiny85 U1
 U 1 1 5ADEF82C
 P 3800 1600
 F 0 "U1" H 3950 1250 60  0000 C CNN
 F 1 "ATTiny85" H 3750 2000 60  0000 C CNN
-F 2 "Housings_DIP:DIP-8_W7.62mm_Socket" H 3850 1300 60  0001 C CNN
+F 2 "Housings_QFP:TQFP-44_10x10mm_Pitch0.8mm" H 3850 1300 60  0001 C CNN
 F 3 "" H 3850 1300 60  0001 C CNN
 	1    3800 1600
@@
 $EndComp
 $Comp
-L SSD1306_OLED U2
+L Custom-Library:SSD1306_OLED U2
 U 1 1 5ADEF917
 P 4200 3200
@@
 $EndComp
 $Comp
-L Speaker LS1
+L Device:Speaker LS1
 U 1 1 5ADEFA7E
 P 5300 1800
@@
 $EndComp
 $Comp
-L C C0
+L Device:C C0
 U 1 1 5ADEFBB3
 P 5500 2850
@@
 $EndComp
 $Comp
-L R R10
+L Device:R R10
 U 1 1 5ADEFD2B
 P 5500 3050
@@
 $EndComp
 $Comp
-L D_ALT D0
+L Device:D_ALT D0
 U 1 1 5ADEFD9E
 P 5500 3350
@@
 $EndComp
 $Comp
-L SW_Push SW1
+L switches:SW_Push SW1
 U 1 1 5ADF012F
 P 2350 3400
@@
 $EndComp
 $Comp
-L SW_Push SW2
+L switches:SW_Push SW2
 U 1 1 5ADF0194
 P 2350 3800
@@
 $EndComp
 $Comp
-L SW_Push SW3
+L switches:SW_Push SW3
 U 1 1 5ADF01EB
 P 2350 4250
@@
 $EndComp
 $Comp
-L SW_Push SW4
+L switches:SW_Push SW4
 U 1 1 5ADF0255
 P 2350 4700
@@
 $EndComp
 $Comp
-L SW_Push SW5
+L switches:SW_Push SW5
 U 1 1 5ADF02A9
 P 2350 5100
@@
 $EndComp
 $Comp
-L SW_Push SW6
+L switches:SW_Push SW6
 U 1 1 5ADF02FB
 P 2350 5500
@@
 $EndComp
 $Comp
-L SW_Push SW7
+L switches:SW_Push SW7
 U 1 1 5ADF0346
 P 2350 5900
@@
 $EndComp
 $Comp
-L R R1
+L Device:R R1
 U 1 1 5ADF05B6
 P 2950 3400
@@
 $EndComp
 $Comp
-L R R2
+L Device:R R2
 U 1 1 5ADF0637
 P 2950 3800
@@
 $EndComp
 $Comp
-L R R3
+L Device:R R3
 U 1 1 5ADF068B
 P 2950 4250
@@
 $EndComp
 $Comp
-L R R4
+L Device:R R4
 U 1 1 5ADF06E2
 P 2950 4700
@@
 $EndComp
 $Comp
-L R R5
+L Device:R R5
 U 1 1 5ADF073C
 P 2950 5100
@@
 $EndComp
 $Comp
-L R R6
+L Device:R R6
 U 1 1 5ADF079F
 P 2950 5500
@@
 $EndComp
 $Comp
-L R R7
+L Device:R R7
 U 1 1 5ADF07FD
 P 2950 5900
@@
 $EndComp
 $Comp
-L R R9
+L Device:R R9
 U 1 1 5ADF1316
 P 3750 4700
@@
 $EndComp
 $Comp
-L SW_Push SW0
+L switches:SW_Push SW0
 U 1 1 5ADF1FBC
 P 2700 1300
@@
 $EndComp
 $Comp
-L C C1
+L Device:C C1
 U 1 1 5ADF20D8
 P 4250 1050
@@
 $EndComp
 $Comp
-L GND #PWR01
+L power:GND #PWR01
 U 1 1 5ADF25F0
 P 3350 1950
@@
 $EndComp
 $Comp
-L GND #PWR02
+L power:GND #PWR02
 U 1 1 5ADF2A2D
 P 1750 2850
@@
 $EndComp
 $Comp
-L GND #PWR03
+L power:GND #PWR03
 U 1 1 5ADF2E03
 P 4750 3000
@@
 $EndComp
 $Comp
-L GND #PWR04
+L power:GND #PWR04
 U 1 1 5ADF2E6B
 P 3600 3150
@@
 $EndComp
 $Comp
-L GND #PWR05
+L power:GND #PWR05
 U 1 1 5ADF3429
 P 5950 2850
@@
 $EndComp
 $Comp
-L GND #PWR06
+L power:GND #PWR06
 U 1 1 5ADFE45B
 P 2450 1400
@@
 $EndComp
 $Comp
-L GND #PWR07
+L power:GND #PWR07
 U 1 1 5AE00125
 P 4100 4700
@@
 $EndComp
 $Comp
-L GND #PWR08
+L power:GND #PWR08
 U 1 1 5ADF2588
 P 4650 900
@@
 $EndComp
 $Comp
-L SW_DIP_x01 SW8
+L switches:SW_DIP_x01 SW8
 U 1 1 5B17B9FC
 P 2050 2000
@@
 $EndComp
 $Comp
-L +3.3V #PWR09
+L power:+3.3V #PWR09
 U 1 1 5B17C77C
 P 4650 1350
@@
 $EndComp
 $Comp
-L +3.3V #PWR010
+L power:+3.3V #PWR010
 U 1 1 5B17C81F
 P 6150 3350
@@
 $EndComp
 $Comp
-L +3.3V #PWR011
+L power:+3.3V #PWR011
 U 1 1 5B17C8E4
 P 1550 4350
@@
 $EndComp
 $Comp
-L +3.3V #PWR012
+L power:+3.3V #PWR012
 U 1 1 5B17C932
 P 2500 2000
@@
 $EndComp
 $Comp
-L +3.3V #PWR013
+L power:+3.3V #PWR013
 U 1 1 5B17D029
 P 4000 2700
@@
 $EndComp
 $Comp
-L GND #PWR014
+L power:GND #PWR014
 U 1 1 5B17D456
 P 5100 2150
@@
 $EndComp
 $Comp
-L Battery_Cell BT1
+L Device:Battery_Cell BT1
 U 1 1 5B17BFB1
 P 1750 2600
@@
 $EndComp
 $Comp
-L C C2
+L Device:C C2
 U 1 1 5B30B920
 P 3700 2850
@@
 	4300 3000 4300 2850
 Wire Wire Line
-	4300 2850 5350 2850
+	4300 2850 4900 2850
 Wire Wire Line
 	5650 2850 5950 2850
@@
 	5350 3050 5150 3050
 Wire Wire Line
-	5150 2850 5150 3350
+	5150 2850 5150 3050
 Connection ~ 5150 2850
 Wire Wire Line
@@
 	5800 3050 5800 3350
 Wire Wire Line
-	5650 3350 6150 3350
+	5650 3350 5800 3350
 Wire Wire Line
 	5150 3350 5350 3350
@@
 	4900 850  4900 2850
 Wire Wire Line
-	2900 1300 3350 1300
+	2900 1300 3100 1300
 Wire Wire Line
 	3350 1300 3350 1350
@@
 Wire Wire Line
 	1800 3800 2150 3800
-Connection ~ 1800 3400
 Wire Wire Line
 	1800 4250 2150 4250
@@
 	3400 5900 3100 5900
 Wire Wire Line
-	3400 3150 3400 5900
-Wire Wire Line
-	3100 4700 3600 4700
+	3400 3150 3400 3400
+Wire Wire Line
+	3100 4700 3400 4700
 Wire Wire Line
 	3100 5500 3400 5500
@@
 	3100 850  4900 850
 Wire Wire Line
-	1800 3400 1800 5900
+	1800 3400 1800 3800
 Wire Wire Line
 	3400 3150 3100 3150
@@
 	1550 4500 1550 4350
 Wire Wire Line
-	4250 1350 4650 1350
+	4250 1350 4400 1350
 Wire Wire Line
 	4250 1800 5100 1800
@@
 	2350 2000 2500 2000
 Wire Wire Line
-	4000 2700 4000 3000
+	4000 2700 4000 2850
 Wire Wire Line
 	4000 2850 3850 2850
 Connection ~ 4000 2850
 Wire Wire Line
-	3550 3000 3900 3000
+	3550 3000 3600 3000
 Wire Wire Line
 	3600 3000 3600 3150
@@
 	3550 2850 3550 3000
 Connection ~ 3600 3000
+Wire Wire Line
+	5150 2850 5350 2850
+Wire Wire Line
+	5150 3050 5150 3350
+Wire Wire Line
+	5800 3350 6150 3350
+Wire Wire Line
+	4900 2850 5150 2850
+Wire Wire Line
+	3100 1300 3350 1300
+Wire Wire Line
+	1800 3800 1800 4250
+Wire Wire Line
+	1800 4250 1800 4500
+Wire Wire Line
+	1800 4700 1800 5100
+Wire Wire Line
+	1800 5100 1800 5500
+Wire Wire Line
+	1800 5500 1800 5900
+Wire Wire Line
+	3400 5500 3400 5900
+Wire Wire Line
+	3400 5100 3400 5500
+Wire Wire Line
+	3400 4700 3400 5100
+Wire Wire Line
+	3400 4700 3600 4700
+Wire Wire Line
+	3400 4250 3400 4700
+Wire Wire Line
+	3400 3800 3400 4250
+Wire Wire Line
+	3400 3400 3400 3800
+Wire Wire Line
+	1800 4500 1800 4700
+Wire Wire Line
+	4400 1350 4650 1350
+Wire Wire Line
+	4000 2850 4000 3000
+Wire Wire Line
+	3600 3000 3900 3000
 $EndSCHEMATC
