File: board/scroll/scroll.sch (KiCad schematic (older format))
At the start: 2 parts

Commit message: schematic annotations
Parts:
- gave numbers to parts that had none: 2
Changed lines of the file:
@@
 $EndDescr
 $Comp
-L Custom~Library:ATTiny85 U?
+L Custom~Library:ATTiny85 U1
 U 1 1 5BBF0469
 P 4550 3900
-F 0 "U?" H 4550 4437 60  0000 C CNN
+F 0 "U1" H 4550 4437 60  0000 C CNN
 F 1 "ATTiny85" H 4550 4331 60  0000 C CNN
 F 2 "Housings_DIP:DIP-8_W7.62mm" H 4600 3600 60  0001 C CNN
@@
 $EndComp
 $Comp
-L Connector:AVR-ISP-6 J?
+L Connector:AVR-ISP-6 J1
 U 1 1 5BBF0507
 P 6850 3900
-F 0 "J?" H 6570 3996 50  0000 R CNN
+F 0 "J1" H 6570 3996 50  0000 R CNN
 F 1 "AVR-ISP-6" H 6570 3905 50  0000 R CNN
 F 2 "Custom Footprints:6-pin-prog" V 6600 3950 50  0001 C CNN
@@
 RESET
 $Comp
-L power:+3.3V #PWR?
+L power:+3.3V #PWR0101
 U 1 1 5BBF0720
 P 5150 3650
-F 0 "#PWR?" H 5150 3500 50  0001 C CNN
+F 0 "#PWR0101" H 5150 3500 50  0001 C CNN
 F 1 "+3.3V" H 5165 3823 50  0000 C CNN
 F 2 "" H 5150 3650 50  0001 C CNN
@@
 $EndComp
 $Comp
-L power:GND #PWR?
+L power:GND #PWR0102
 U 1 1 5BBF074D
 P 4000 4150
-F 0 "#PWR?" H 4000 3900 50  0001 C CNN
+F 0 "#PWR0102" H 4000 3900 50  0001 C CNN
 F 1 "GND" H 4005 3977 50  0000 C CNN
 F 2 "" H 4000 4150 50  0001 C CNN
@@
 	7250 4000 7350 4000
 $Comp
-L power:GND #PWR?
+L power:GND #PWR0103
 U 1 1 5BBF0AD6
 P 6750 4300
-F 0 "#PWR?" H 6750 4050 50  0001 C CNN
+F 0 "#PWR0103" H 6750 4050 50  0001 C CNN
 F 1 "GND" H 6755 4127 50  0000 C CNN
 F 2 "" H 6750 4300 50  0001 C CNN
@@
 $EndComp
 $Comp
-L power:+3.3V #PWR?
+L power:+3.3V #PWR0104
 U 1 1 5BBF0AE5
 P 6750 3400
-F 0 "#PWR?" H 6750 3250 50  0001 C CNN
+F 0 "#PWR0104" H 6750 3250 50  0001 C CNN
 F 1 "+3.3V" H 6765 3573 50  0000 C CNN
 F 2 "" H 6750 3400 50  0001 C CNN
