File: board/upgrade/ArchMage.kicad_pcb (KiCad board)
At the start: 2 copper layers, 15.5 x 21 mm, 3 parts, among them J1 Conn_02x03_Counter_Clockwise, J2 Conn_02x04_Counter_Clockwise, U1 ATmega1284P-AU

Commit message: changes that I've forgotten now
Parts:
- J1: value Conn_02x03_Counter_Clockwise -> ISP; footprint Custom Footprints:6-pin-prog -> Pin_Headers:Pin_Header_Straight_2x03_Pitch2.54mm
- J2: value Conn_02x04_Counter_Clockwise -> DIP8; footprint Custom Footprints:DIP-8_W7.62mm -> Housings_DIP:DIP-8_W7.62mm
- moved J1 0.71 mm to (158.8, 85.2), turned to 90 degrees
Connections:
- J1 pad 1: GND -> MISO
- J1 pad 3: RESET -> SCK
- J1 pad 5: MISO -> RESET
- J1 pad 6: SCK -> GND
Routing:
- net MOSI: track 12.6 -> 0.00 mm
- net AD2: track 10.6 -> 0.00 mm, vias 1 -> 0
- net RESET: track 10.4 -> 0.00 mm, vias 1 -> 0
- net PB3: track 10.3 -> 0.00 mm
- net MISO: track 9.79 -> 0.00 mm
- net Vcc: track 9.20 -> 0.00 mm
- net GND: track 9.16 -> 0.00 mm
- net PB0: track 9.01 -> 0.00 mm
- net PB1: track 6.45 -> 0.00 mm, vias 1 -> 0
- net SCK: track 5.89 -> 0.00 mm
- net PB2: track 2.33 -> 0.00 mm
Other:
- board text removed: "+"
- board text removed: "-"
- board text removed: "c"
- board text removed: "i"
- board text removed: "o"
- board text removed: "r"
